Commit message: Add files

File: orne_box_description/urdf/orne_box.gazebo.xacro (robot description, xacro)
@@ -40,4 +40,49 @@
     <material>Gazebo/White</material>
   </gazebo>
+  <joint name="camera_rgb_joint" type="fixed">
+    <parent link="base_link"/>
+    <child link="camera_rgb_optical_frame"/>
+    <origin xyz="-0.08 0.0 0.8" rpy="0 -0.05 0"/>
+  </joint>
+  <link name="camera_rgb_optical_frame"/>
+  <gazebo reference="camera_rgb_optical_frame">
+    <sensor type="camera" name="camera1">
+      <always_on>true</always_on>
+      <update_rate>30</update_rate>
+      <visualize>true</visualize>
+      <camera name="head">
+        <horizontal_fov>1.571</horizontal_fov>
+        <image>
+          <width>640</width>
+          <height>480</height>
+          <format>R8G8B8</format>
+        </image>
+        <clip>
+          <near>0.03</near>
+          <far>100</far>
+        </clip>
+        <noise>
+          <type>gaussian</type>
+          <mean>0.0</mean>
+          <stddev>0.007</stddev>
+        </noise>
+      </camera>
+      <plugin name="camera_controller" filename="libgazebo_ros_camera.so">
+        <!-- <topicName>camera_right</topicName> -->
+        <alwaysOn>true</alwaysOn>
+        <updateRate>30.0</updateRate>
+        <cameraName>camera</cameraName>
+        <frameName>camera_rgb_optical_frame</frameName>
+        <imageTopicName>image_raw</imageTopicName>
+        <cameraInfoTopicName>/camera_info</cameraInfoTopicName>
+        <hackBaseline>0.07</hackBaseline>
+        <distortionK1>0.0</distortionK1>
+        <distortionK2>0.0</distortionK2>
+        <distortionK3>0.0</distortionK3>
+        <distortionT1>0.0</distortionT1>
+        <distortionT2>0.0</distortionT2>
+      </plugin>
+    </sensor>
+  </gazebo>
   <!-- @TODO More clear boolean operation -->
   <xacro:if value="${'$(arg ignition_gazebo)' == 'false'}">
@@ -60,5 +105,5 @@
     <!-- hokuyo -->
     <gazebo reference="hokuyo_link">
-      <sensor type="ray" name="head_hokuyo_sensor">
+      <sensor type="gpu_ray" name="head_hokuyo_sensor">
         <pose>0 0 0 0 0 0</pose>
         <visualize>$(arg laser_visual)</visualize>
@@ -92,5 +137,5 @@
           </noise>
         </ray>
-        <plugin name="gazebo_ros_head_hokuyo_controller" filename="libgazebo_ros_laser.so">
+        <plugin name="gazebo_ros_head_hokuyo_controller" filename="libgazebo_ros_gpu_laser.so">
           <topicName>/scan</topicName>
           <frameName>hokuyo_link</frameName>

Commit message: Update

File: orne_box_description/urdf/orne_box.gazebo.xacro (robot description, xacro)
@@ -39,4 +39,49 @@
     <maxVel>1.0</maxVel>
     <material>Gazebo/White</material>
+  </gazebo>
+  <joint name="rfans_camera_rgb_joint" type="fixed">
+    <parent link="base_link"/>
+    <child link="rfans_camera_rgb_optical_frame"/>
+    <origin xyz="0.23 0.0 0.8" rpy="0 -0.05 0"/>
+  </joint>
+  <link name="rfans_camera_rgb_optical_frame"/>
+  <gazebo reference="rfans_camera_rgb_optical_frame">
+    <sensor type="camera" name="camera2">
+      <always_on>false</always_on>
+      <update_rate>30</update_rate>
+      <visualize>false</visualize>
+      <camera name="rfans_head">
+        <horizontal_fov>1.571</horizontal_fov>
+        <image>
+          <width>640</width>
+          <height>480</height>
+          <format>R8G8B8</format>
+        </image>
+        <clip>
+          <near>0.03</near>
+          <far>100</far>
+        </clip>
+        <noise>
+          <type>gaussian</type>
+          <mean>0.0</mean>
+          <stddev>0.007</stddev>
+        </noise>
+      </camera>
+      <plugin name="rfans_camera_controller" filename="libgazebo_ros_camera.so">
+        <!-- <topicName>camera_right</topicName> -->
+        <alwaysOn>false</alwaysOn>
+        <updateRate>30.0</updateRate>
+        <cameraName>rfans_camera</cameraName>
+        <frameName>camera_rgb_optical_frame</frameName>
+        <imageTopicName>image_raw</imageTopicName>
+        <cameraInfoTopicName>/camera_info</cameraInfoTopicName>
+        <hackBaseline>0.07</hackBaseline>
+        <distortionK1>0.0</distortionK1>
+        <distortionK2>0.0</distortionK2>
+        <distortionK3>0.0</distortionK3>
+        <distortionT1>0.0</distortionT1>
+        <distortionT2>0.0</distortionT2>
+      </plugin>
+    </sensor>
   </gazebo>
   <joint name="camera_rgb_joint" type="fixed">

Commit message: Add omni camera

File: orne_box_description/urdf/orne_box.gazebo.xacro (robot description, xacro)
@@ -39,4 +39,179 @@
     <maxVel>1.0</maxVel>
     <material>Gazebo/White</material>
+  </gazebo>
+  <gazebo reference="omnidirectional_camera_front_frame">
+      <sensor type="wideanglecamera" name="camera">
+        <camera>
+          <horizontal_fov>3.14</horizontal_fov>
+          <image>
+            <width>640</width>
+            <height>640</height>
+          </image>
+          <clip>
+            <near>0.1</near>
+            <far>50</far>
+          </clip>
+          <lens>
+            <!-- <type>gnomonical</type> -->
+            <type>custom</type>
+            <custom_function>
+              <c1>0.5</c1>
+              <c2>4.0</c2>
+              <f>1.0</f>
+              <fun>cos</fun>
+            </custom_function>
+            <scale_to_hfov>true</scale_to_hfov>
+            <cutoff_angle>3.14</cutoff_angle>
+            <env_texture_size>512</env_texture_size>
+          </lens>
+        </camera>
+        <plugin name="camera_controller" filename="libgazebo_ros_camera.so">
+        <alwaysOn>true</alwaysOn>
+        <updateRate>10.0</updateRate>
+        <cameraName>camera</cameraName>
+        <frameName>camera_rgb_optical_front_frame</frameName>
+        <imageTopicName>rgb/image_raw_front</imageTopicName>
+        <cameraInfoTopicName>rgb/camera_info</cameraInfoTopicName>
+        <CxPrime></CxPrime>
+        <Cx></Cx>
+        <Cy></Cy>
+        <focalLength></focalLength>
+        <hackBaseline>0.7</hackBaseline>
+        <distortionK1>0.0</distortionK1>
+        <distortionK2>0.0</distortionK2>
+        <distortionK3>0.0</distortionK3>
+        <distortionT1>0.0</distortionT1>
+        <distortionT2>0.0</distortionT2>
+      </plugin>
+      </sensor>
+  </gazebo>
+  <joint name="omni_camera_joint" type="fixed">
+    <origin xyz="0.23 0 0.6" rpy="0 0 0"/>
+    <parent link="base_link"/>
+    <child link="camera_link"/>
+  </joint>
+  <link name="camera_link">
+    <collision>
+      <origin xyz="0 0 0" rpy="0 0 0"/>
+      <geometry>
+        <box size="0.015 0.030 0.027"/>
+      </geometry>
+    </collision>
+  </link>
+  <joint name="camera_rgb_front_joint" type="fixed">
+    <origin xyz="0 0 0" rpy="1.57 0 0"/>
+    <parent link="camera_link"/>
+    <child link="omnidirectional_camera_front_frame"/>
+  </joint>
+  <link name="omnidirectional_camera_front_frame"/>
+  <joint name="camera_rgb_optical_front_joint" type="fixed">
+    <origin xyz="0 0 0" rpy="0 0 0"/>
+    <parent link="omnidirectional_camera_front_frame"/>
+    <child link="camera_rgb_optical_front_frame"/>
+  </joint>
+  <link name="camera_rgb_optical_front_frame"/>
+  <joint name="camera_rgb_back_joint" type="fixed">
+    <origin xyz="0 0 0" rpy="-1.57 0 3.14"/>
+    <parent link="camera_link"/>
+    <child link="omnidirectional_camera_back_frame"/>
+  </joint>
+  <link name="omnidirectional_camera_back_frame"/>
+  <joint name="camera_rgb_optical_back_joint" type="fixed">
+    <origin xyz="0 0 0" rpy="0 0 0"/>
+    <parent link="omnidirectional_camera_back_frame"/>
+    <child link="camera_rgb_optical_back_frame"/>
+  </joint>
+  <link name="camera_rgb_optical_back_frame"/>
+  <gazebo reference="omnidirectional_camera_front_frame">
+      <sensor type="wideanglecamera" name="camera">
+        <camera>
+          <horizontal_fov>3.14</horizontal_fov>
+          <image>
+            <width>640</width>
+            <height>640</height>
+          </image>
+          <clip>
+            <near>0.1</near>
+            <far>50</far>
+          </clip>
+          <lens>
+            <!-- <type>gnomonical</type> -->
+            <type>custom</type>
+            <custom_function>
+              <c1>0.5</c1>
+              <c2>4.0</c2>
+              <f>1.0</f>
+              <fun>cos</fun>
+            </custom_function>
+            <scale_to_hfov>true</scale_to_hfov>
+            <cutoff_angle>3.14</cutoff_angle>
+            <env_texture_size>512</env_texture_size>
+          </lens>
+        </camera>
+        <plugin name="camera_controller" filename="libgazebo_ros_camera.so">
+        <alwaysOn>true</alwaysOn>
+        <updateRate>10.0</updateRate>
+        <cameraName>camera</cameraName>
+        <frameName>camera_rgb_optical_front_frame</frameName>
+        <imageTopicName>rgb/image_raw_front</imageTopicName>
+        <cameraInfoTopicName>rgb/camera_info</cameraInfoTopicName>
+        <CxPrime></CxPrime>
+        <Cx></Cx>
+        <Cy></Cy>
+        <focalLength></focalLength>
+        <hackBaseline>0.7</hackBaseline>
+        <distortionK1>0.0</distortionK1>
+        <distortionK2>0.0</distortionK2>
+        <distortionK3>0.0</distortionK3>
+        <distortionT1>0.0</distortionT1>
+        <distortionT2>0.0</distortionT2>
+      </plugin>
+      </sensor>
+  </gazebo>
+  <gazebo reference="omnidirectional_camera_back_frame">
+      <sensor type="wideanglecamera" name="camera">
+        <camera>
+          <horizontal_fov>3.14</horizontal_fov>
+          <image>
+            <width>640</width>
+            <height>640</height>
+          </image>
+          <clip>
+            <near>0.1</near>
+            <far>50</far>
+          </clip>
+          <lens>
+            <!-- <type>gnomonical</type> -->
+            <type>custom</type>
+            <custom_function>
+              <c1>0.5</c1>
+              <c2>4.0</c2>
+              <f>1.0</f>
+              <fun>cos</fun>
+            </custom_function>
+            <scale_to_hfov>true</scale_to_hfov>
+            <cutoff_angle>3.14</cutoff_angle>
+            <env_texture_size>512</env_texture_size>
+          </lens>
+        </camera>
+        <plugin name="camera_controller" filename="libgazebo_ros_camera.so">
+        <alwaysOn>true</alwaysOn>
+        <updateRate>10.0</updateRate>
+        <cameraName>camera</cameraName>
+        <frameName>camera_rgb_optical_back_frame</frameName>
+        <imageTopicName>rgb/image_raw_back</imageTopicName>
+        <cameraInfoTopicName>rgb/camera_info</cameraInfoTopicName>
+        <CxPrime></CxPrime>
+        <Cx></Cx>
+        <Cy></Cy>
+        <focalLength></focalLength>
+        <hackBaseline>0.7</hackBaseline>
+        <distortionK1>0.0</distortionK1>
+        <distortionK2>0.0</distortionK2>
+        <distortionK3>0.0</distortionK3>
+        <distortionT1>0.0</distortionT1>
+        <distortionT2>0.0</distortionT2>
+      </plugin>
+      </sensor>
   </gazebo>
   <joint name="rfans_camera_rgb_joint" type="fixed">

File: orne_box_description/urdf/orne_box_3d_lidar.urdf.xacro (robot description, xacro)
@@ -6,8 +6,11 @@
   <xacro:if value="${'$(arg ignition_gazebo)' == 'false'}">
     <xacro:include filename="$(find velodyne_description)/urdf/VLP-16.urdf.xacro"/>
-    <!-- Setting for 3D-LiDAR -->
     <xacro:VLP-16 parent="base_link" name="surestar" topic="/rfans_points" organize_cloud="false" hz="10" samples="440" gpu="true">
       <origin xyz="0.23 0 0.40" rpy="0 0 0"/>
     </xacro:VLP-16>
+    <!-- <xacro:include filename="$(find velodyne_description)/urdf/HDL-32E.urdf.xacro"/>
+    <xacro:HDL-32E parent="base_link" name="surestar" topic="/rfans_points" organize_cloud="false" hz="10" samples="440" gpu="true">
+      <origin xyz="0.23 0 0.40" rpy="0 0 0"/>
+    </xacro:HDL-32E> -->
   </xacro:if>
   <xacro:if value="$(arg ignition_gazebo)">
